Commit message: lidar and camera added - color done

File: Project2-Go-Chase-It/catkin_ws/src/my_robot/urdf/my_robot.xacro (robot description, xacro)
@@ -55,4 +55,7 @@
     </visual>
   </link>
+  <gazebo reference="chassis">
+    <material>Gazebo/Green</material>
+  </gazebo>
   <link name='left_wheel'>
     <visual name='left_wheel_visual'>
@@ -78,4 +81,7 @@
     </inertial>
   </link>
+  <gazebo reference="left_wheel">
+    <material>Gazebo/DarkGray</material>
+  </gazebo>
   <joint type="continuous" name="left_wheel_hinge">
     <origin xyz="0 0.15 0" rpy="0 0 0"/>
@@ -92,4 +98,5 @@
         <cylinder radius="0.1" length="0.05"/>
       </geometry>
+      <!-- <material>Gazebo/Green</material> -->
     </visual>
     <collision name='right_wheel_collision'>
@@ -109,11 +116,76 @@
     </inertial>
   </link>
-<joint type="continuous" name="right_wheel_hinge">
-  <origin xyz="0 -0.15 0" rpy="0 0 0"/>
-  <child link="right_wheel"/>
-  <parent link="chassis"/>
-  <axis xyz="0 1 0" rpy="0 0 0"/>
-  <limit effort="10000" velocity="1000"/>
-  <dynamics damping="1.0" friction="1.0"/>
-</joint>
+  <gazebo reference="right_wheel">
+    <material>Gazebo/DarkGray</material>
+  </gazebo>
+  <joint type="continuous" name="right_wheel_hinge">
+    <origin xyz="0 -0.15 0" rpy="0 0 0"/>
+    <child link="right_wheel"/>
+    <parent link="chassis"/>
+    <axis xyz="0 1 0" rpy="0 0 0"/>
+    <limit effort="10000" velocity="1000"/>
+    <dynamics damping="1.0" friction="1.0"/>
+  </joint>
+  <link name='camera'>
+    <visual name='camera_visual'>
+      <origin xyz="0 0 0" rpy=" 0 0 0"/>
+      <geometry>
+        <box size="0.05 0.05 0.05"/>
+      </geometry>
+    </visual>
+    <collision name='camera_collision'>
+      <origin xyz="0 0 0" rpy=" 0 0 0"/>
+      <geometry>
+        <box size="0.05 0.05 0.05"/>
+      </geometry>
+    </collision>
+    <inertial>
+      <mass value="0.1"/>
+      <origin xyz="0.0 0 0" rpy=" 0 0 0"/>
+      <inertia
+          ixx="1e-6" ixy="0" ixz="0"
+          iyy="1e-6" iyz="0"
+          izz="1e-6"
+      />
+    </inertial>
+  </link>
+  <gazebo reference="camera">
+    <material>Gazebo/Orange</material>
+  </gazebo>
+  <joint type="fixed" name="camera_joint">
+    <origin xyz="0.2 0 0" rpy="0 0 0"/>
+    <child link="camera"/>
+    <parent link="chassis"/>
+    <axis xyz="0 1 0" rpy="0 0 0"/>
+  </joint>
+  <link name='hokuyo'>
+    <visual name='hokuyo_visual'>
+      <origin xyz="0 0 0" rpy=" 0 0 0"/>
+      <geometry>
+        <!-- <box size="0.1 0.1 0.1"/> -->
+        <mesh filename="package://my_robot/meshes/hokuyo.dae"/>
+      </geometry>
+    </visual>
+    <collision name='hokuyo_collision'>
+      <origin xyz="0 0 0" rpy=" 0 0 0"/>
+      <geometry>
+        <box size="0.1 0.1 0.1"/>
+      </geometry>
+    </collision>
+    <inertial>
+      <mass value="1e-5"/>
+      <origin xyz="0.0 0 0" rpy=" 0 0 0"/>
+      <inertia
+          ixx="1e-6" ixy="0" ixz="0"
+          iyy="1e-6" iyz="0"
+          izz="1e-6"
+      />
+    </inertial>
+  </link>
+  <joint type="fixed" name="hokuyo_joint">
+    <origin xyz="0.15 0 0.1" rpy="0 0 0"/>
+    <child link="hokuyo"/>
+    <parent link="chassis"/>
+    <axis xyz="0 1 0" rpy="0 0 0"/>
+  </joint>
 </robot>

Commit message: dimensions of robot changed

File: Project2-Go-Chase-It/catkin_ws/src/my_robot/urdf/my_robot.xacro (robot description, xacro)
@@ -1,4 +1,5 @@
 <?xml version='1.0'?>
 <robot name="my_robot" xmlns:xacro="http://www.ros.org/wiki/xacro">
+  <xacro:include filename="$(find my_robot)/urdf/my_robot.gazebo" />
   <link name="robot_footprint"></link>
   <joint name="robot_footprint_joint" type="fixed">
@@ -21,5 +22,5 @@
       <origin xyz="0 0 0" rpy=" 0 0 0"/>
       <geometry>
-        <box size=".4 .2 .1"/>
+        <box size=".4 .25 .1"/>
       </geometry>
     </collision>
@@ -27,5 +28,5 @@
       <origin xyz="0 0 0" rpy=" 0 0 0"/>
       <geometry>
-        <box size=".4 .2 .1"/>
+        <box size=".4 .25 .1"/>
       </geometry>
     </visual>
@@ -62,5 +63,5 @@
       <origin xyz="0 0 0" rpy=" 0 1.5707 1.5707"/>
       <geometry>
-        <cylinder radius="0.1" length="0.05"/>
+        <cylinder radius="0.11" length="0.05"/>
       </geometry>
     </visual>
@@ -68,5 +69,5 @@
       <origin xyz="0 0 0" rpy=" 0 1.5707 1.5707"/>
       <geometry>
-        <cylinder radius="0.1" length="0.05"/>
+        <cylinder radius="0.11" length="0.05"/>
       </geometry>
     </collision>
@@ -96,5 +97,5 @@
       <origin xyz="0 0 0" rpy=" 0 1.5707 1.5707"/>
       <geometry>
-        <cylinder radius="0.1" length="0.05"/>
+        <cylinder radius="0.11" length="0.05"/>
       </geometry>
       <!-- <material>Gazebo/Green</material> -->
@@ -103,5 +104,5 @@
       <origin xyz="0 0 0" rpy=" 0 1.5707 1.5707"/>
       <geometry>
-        <cylinder radius="0.1" length="0.05"/>
+        <cylinder radius="0.11" length="0.05"/>
       </geometry>
     </collision>
@@ -184,5 +185,5 @@
   </link>
   <joint type="fixed" name="hokuyo_joint">
-    <origin xyz="0.15 0 0.1" rpy="0 0 0"/>
+    <origin xyz="0.15 0 0.09" rpy="0 0 0"/>
     <child link="hokuyo"/>
     <parent link="chassis"/>

Commit message: dimensions of robot changed again, project 1 world added

File: Project2-Go-Chase-It/catkin_ws/src/my_robot/urdf/my_robot.xacro (robot description, xacro)
@@ -22,5 +22,5 @@
       <origin xyz="0 0 0" rpy=" 0 0 0"/>
       <geometry>
-        <box size=".4 .25 .1"/>
+        <box size=".43 .25 .1"/>
       </geometry>
     </collision>
@@ -28,5 +28,5 @@
       <origin xyz="0 0 0" rpy=" 0 0 0"/>
       <geometry>
-        <box size=".4 .25 .1"/>
+        <box size=".43 .25 .1"/>
       </geometry>
     </visual>
@@ -34,5 +34,5 @@
       <origin xyz="-0.15 0 -0.05" rpy=" 0 0 0"/>
       <geometry>
-        <sphere radius="0.0499"/>
+        <sphere radius="0.06"/>
       </geometry>
     </collision>
@@ -40,5 +40,5 @@
       <origin xyz="-0.15 0 -0.05" rpy=" 0 0 0"/>
       <geometry>
-        <sphere radius="0.05"/>
+        <sphere radius="0.06"/>
       </geometry>
     </visual>
@@ -46,5 +46,5 @@
       <origin xyz="0.15 0 -0.05" rpy=" 0 0 0"/>
       <geometry>
-        <sphere radius="0.0499"/>
+        <sphere radius="0.06"/>
       </geometry>
     </collision>
@@ -52,5 +52,5 @@
       <origin xyz="0.15 0 -0.05" rpy=" 0 0 0"/>
       <geometry>
-        <sphere radius="0.05"/>
+        <sphere radius="0.06"/>
       </geometry>
     </visual>
@@ -155,5 +155,5 @@
   </gazebo>
   <joint type="fixed" name="camera_joint">
-    <origin xyz="0.2 0 0" rpy="0 0 0"/>
+    <origin xyz="0.25 0 0" rpy="0 0 0"/>
     <child link="camera"/>
     <parent link="chassis"/>

Commit message: hell lot of changes - chases the ball finally

File: Project2-Go-Chase-It/catkin_ws/src/my_robot/urdf/my_robot.xacro (robot description, xacro)
@@ -91,5 +91,5 @@
     <axis xyz="0 1 0" rpy="0 0 0"/>
     <limit effort="10000" velocity="1000"/>
-    <dynamics damping="1.0" friction="1.0"/>
+    <dynamics damping="0.3" friction="0.3"/>
   </joint>
   <link name='right_wheel'>
@@ -126,5 +126,5 @@
     <axis xyz="0 1 0" rpy="0 0 0"/>
     <limit effort="10000" velocity="1000"/>
-    <dynamics damping="1.0" friction="1.0"/>
+    <dynamics damping="0.3" friction="0.3"/>
   </joint>
   <link name='camera'>
